File: pcb/mailbox-notifier.brd (EAGLE design)
At the start: 35 x 100 mm, 68 parts, among them CON1 3P-SH-SIDE, Q1 AO3401, U1 MCP73832, U10 MIC2019, U11 74LVC1G17, U2 MIC23155, U3 FS312F-G, U4 FS8205, U5 EFM32PG1B200F256GM32, U6 SST26VF016B, U7 RFM69HW, U8 SI7021, U9 MIC2019, X1 40MHz

Commit message: nothing to do
Parts:
- moved R6 12.2 mm to (29.1, 79.2)
- moved R5 8.40 mm to (29.1, 81.1)
Connections:
- net !FLASH_CS: now also U5.14; no longer U5.16
- net !RFM_CS: now also U5.13; no longer U5.14
- net RFM_RST: now also U5.16; no longer U5.13
Routing:
- net !RFM_CS: track 0.00 -> 60.7 mm, vias 0 -> 4
- net US0_MISO: track 0.00 -> 56.2 mm, vias 0 -> 3
- net RFM_RST: track 0.00 -> 54.6 mm, vias 0 -> 3
- net US0_MOSI: track 0.00 -> 50.3 mm, vias 0 -> 3
- net RFM_IRQ: track 0.00 -> 47.5 mm, vias 0 -> 2
- net US0_CLK: track 0.00 -> 45.2 mm, vias 0 -> 3
- net 2V8_PGOOD: track 0.00 -> 43.3 mm, vias 0 -> 3
- net BAT_STAT: track 6.03 -> 47.6 mm, vias 1 -> 3
- net VBAT_SENSE: track 8.52 -> 40.5 mm, vias 0 -> 2
- net !FLASH_CS: track 3.98 -> 35.8 mm, vias 0 -> 2
- net EXT_TRIG: track 0.00 -> 16.5 mm, vias 0 -> 2
- net EXT_EN: track 0.00 -> 10.1 mm, vias 0 -> 2
- net 1V8: track 4.02 -> 5.92 mm
- net VBAT: track 40.9 -> 42.6 mm, vias 3 -> 4
- net SWDIO: track 13.1 -> 13.8 mm
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
Commit message: Finish board Generate gerbers
Parts:
- added LOGO1: GECKO-14MM, Silkscreen:GECKO_14MM
- added LOGO2: OSHW-LOGOM, Silkscreen:OSHW-LOGO-M
Other:
- board text added: "Designed in Portugal"
- board text added: "IoT Mailbox notifier v2 Jun 2019"

Commit message: Machine gun
Routing:
- net GND: vias 6 -> 228

Commit message: Fix USB C
Parts:
- U5: device EFM32:QFN32 -> EFM32:QFN32_0.5P
- USB1: value USB-C-16P-SMD-FLAT-SIDE -> USB-C-16P-SMD-FLAT-SIDE-TYPE-2; device USB Connector:USB-C-16P-SMD-FLAT-SIDE -> USB Connector:USB-C-16P-SMD-FLAT-SIDE-TYPE-2
Connections:
- net GND: now also USB1.A1/B12, USB1.B1/A12; no longer USB1.GND@0, USB1.GND@1
- net N$3: now also USB1.B5; no longer USB1.CC2
- net N$4: now also USB1.A4/B9, USB1.B4/A9; no longer USB1.VBUS@0, USB1.VBUS@1
- net N$5: now also USB1.A5; no longer USB1.CC1
Routing:
- net N$5: track 7.16 -> 7.66 mm
- net N$3: track 7.66 -> 7.16 mm
Changed lines of the file:
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@@
 <setting verticaltext="up"/>
 </settings>
-<grid distance="0.5" unitdist="mm" unit="mm" style="lines" multiple="1" display="yes" altdistance="0.05" altunitdist="mm" altunit="mm"/>
+<grid distance="0.1" unitdist="mm" unit="mm" style="lines" multiple="1" display="yes" altdistance="0.05" altunitdist="mm" altunit="mm"/>
 <layers>
 <layer number="1" name="Top" color="4" fill="1" visible="yes" active="yes"/>
@@
 <attribute name="VALUE" x="30.314" y="89.389" size="0.762" layer="27" font="vector" ratio="10" rot="R180"/>
 </element>
-<element name="U5" library="EFM32" package="QFN32" value="EFM32PG1B200F256GM32" x="17.5" y="52.3" smashed="yes">
+<element name="U5" library="EFM32" package="QFN32_0.5P" value="EFM32PG1B200F256GM32" x="17.5" y="52.3" smashed="yes">
 <attribute name="NAME" x="20.4" y="55.1" size="0.762" layer="25" font="vector" ratio="10"/>
 </element>
@@
 <attribute name="VALUE" x="6.414" y="84.789" size="0.762" layer="27" font="vector" ratio="10" rot="R180"/>
 </element>
-<element name="USB1" library="USB Connector" package="USB-C-16P-SMD-FLAT-SIDE" value="USB-C-16P-SMD-FLAT-SIDE" x="17.5" y="98.6" smashed="yes" rot="R270">
+<element name="USB1" library="USB Connector" package="USB-C-16P-SMD-FLAT-SIDE-TYPE-2" value="USB-C-16P-SMD-FLAT-SIDE-TYPE-2" x="17.5" y="98.6" smashed="yes" rot="R270">
 <attribute name="NAME" x="16.122" y="96.688" size="0.762" layer="25" font="vector" ratio="10"/>
 <attribute name="VALUE" x="10.642" y="100.378" size="0.762" layer="27" font="vector" ratio="10" rot="R270"/>
@@
 <contactref element="USB1" pad="SHIELD@0"/>
 <contactref element="USB1" pad="SHIELD@3"/>
-<contactref element="USB1" pad="GND@1"/>
-<contactref element="USB1" pad="GND@0"/>
+<contactref element="USB1" pad="B1/A12"/>
+<contactref element="USB1" pad="A1/B12"/>
 <contactref element="R3" pad="1"/>
 <contactref element="R1" pad="1"/>
@@
 </signal>
 <signal name="N$3">
-<contactref element="USB1" pad="CC2"/>
+<contactref element="USB1" pad="B5"/>
 <contactref element="R1" pad="2"/>
-<wire x1="10.81915" y1="96.5" x2="15.1" y2="96.5" width="0.2" layer="1"/>
-<wire x1="16.25" y1="95.35" x2="16.25" y2="93.6" width="0.2" layer="1"/>
-<wire x1="15.1" y1="96.5" x2="16.25" y2="95.35" width="0.2" layer="1"/>
+<wire x1="14.6" y1="96.5" x2="10.81915" y2="96.5" width="0.2" layer="1"/>
+<wire x1="15.75" y1="93.6" x2="15.75" y2="95.35" width="0.2" layer="1"/>
+<wire x1="15.75" y1="95.35" x2="14.6" y2="96.5" width="0.2" layer="1"/>
 </signal>
 <signal name="N$4">
-<contactref element="USB1" pad="VBUS@0"/>
-<contactref element="USB1" pad="VBUS@1"/>
+<contactref element="USB1" pad="A4/B9"/>
+<contactref element="USB1" pad="B4/A9"/>
 <contactref element="F1" pad="2"/>
 <wire x1="15.1" y1="93.6" x2="15.1" y2="92.7" width="0.6096" layer="1"/>
@@
 <wire x1="17.7" y1="91.4" x2="17.7" y2="89.972" width="0.6096" layer="1"/>
 <wire x1="17" y1="92.1" x2="17.7" y2="91.4" width="0.6096" layer="1"/>
-<wire x1="19.9" y1="93.6" x2="19.9" y2="92.7" width="0.6096" layer="1"/>
-<wire x1="19.9" y1="92.7" x2="19.3" y2="92.1" width="0.6096" layer="1"/>
+<wire x1="19.3" y1="92.1" x2="19.9" y2="92.7" width="0.6096" layer="1"/>
 <wire x1="19.3" y1="92.1" x2="18.4" y2="92.1" width="0.6096" layer="1"/>
 <wire x1="18.4" y1="92.1" x2="17.7" y2="91.4" width="0.6096" layer="1"/>
+<wire x1="19.9" y1="92.7" x2="19.9" y2="93.6" width="0.6096" layer="1"/>
 </signal>
 <signal name="N$5">
-<contactref element="USB1" pad="CC1"/>
+<contactref element="USB1" pad="A5"/>
 <contactref element="R3" pad="2"/>
-<wire x1="24.18085" y1="96.5" x2="20.4" y2="96.5" width="0.2" layer="1"/>
-<wire x1="19.25" y1="95.35" x2="19.25" y2="93.6" width="0.2" layer="1"/>
-<wire x1="20.4" y1="96.5" x2="19.25" y2="95.35" width="0.2" layer="1"/>
+<wire x1="19.9" y1="96.5" x2="24.18085" y2="96.5" width="0.2" layer="1"/>
+<wire x1="18.75" y1="93.6" x2="18.75" y2="95.35" width="0.2" layer="1"/>
+<wire x1="18.75" y1="95.35" x2="19.9" y2="96.5" width="0.2" layer="1"/>
 </signal>
 <signal name="EXT_TRIG">
