File: pcb/mailbox-notifier.sch (EAGLE design)
At the start: 68 parts, among them CON1 3P-SH-SIDE, Q1 AO3401, U1 MCP73832, U10 MIC2019, U11 74LVC1G17, U2 MIC23155, U3 FS312F-G, U4 FS8205, U5 EFM32PG1B200F256GM32, U6 SST26VF016B, U7 RFM69HW, U8 SI7021, U9 MIC2019, X1 40MHz

Commit message: nothing to do
Connections:
- net !FLASH_CS: now also U5.PD13; no longer U5.PD15
- net !RFM_CS: now also U5.PD12; no longer U5.PD13
- net RFM_RST: now also U5.PD15; no longer U5.PD12
Changed lines of the file:
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@@
 <?xml version="1.0" encoding="utf-8"?>
 <!DOCTYPE eagle SYSTEM "eagle.dtd">
-<eagle version="9.3.2">
+<eagle version="9.3.0">
 <drawing>
 <settings>
@@
 </segment>
 <segment>
-<label x="175.26" y="132.08" size="1.778" layer="95" xref="yes"/>
-<wire x1="170.18" y1="132.08" x2="175.26" y2="132.08" width="0.1524" layer="91"/>
-<pinref part="U5" gate="G$1" pin="PD15"/>
+<label x="175.26" y="137.16" size="1.778" layer="95" xref="yes"/>
+<wire x1="170.18" y1="137.16" x2="175.26" y2="137.16" width="0.1524" layer="91"/>
+<pinref part="U5" gate="G$1" pin="PD13"/>
 </segment>
 </net>
@@
 </segment>
 </net>
+<net name="US1_CLK" class="0">
+<segment>
+<label x="121.92" y="210.82" size="1.778" layer="95" rot="R180" xref="yes"/>
+<wire x1="127" y1="210.82" x2="121.92" y2="210.82" width="0.1524" layer="91"/>
+<pinref part="U5" gate="G$1" pin="PA1"/>
+</segment>
+</net>
+<net name="US1_MOSI" class="0">
+<segment>
+<label x="96.52" y="213.36" size="1.778" layer="95" rot="R180" xref="yes"/>
+<wire x1="127" y1="213.36" x2="96.52" y2="213.36" width="0.1524" layer="91"/>
+<pinref part="U5" gate="G$1" pin="PA0"/>
+</segment>
+</net>
+<net name="LED_EN" class="0">
+<segment>
+<wire x1="170.18" y1="185.42" x2="175.26" y2="185.42" width="0.1524" layer="91"/>
+<label x="175.26" y="185.42" size="1.778" layer="95" xref="yes"/>
+<pinref part="U5" gate="G$1" pin="PB11"/>
+</segment>
+</net>
+<net name="VBAT_SENSE" class="0">
+<segment>
+<wire x1="127" y1="142.24" x2="121.92" y2="142.24" width="0.1524" layer="91"/>
+<label x="121.92" y="142.24" size="1.778" layer="95" rot="R180" xref="yes"/>
+<pinref part="U5" gate="G$1" pin="PC11"/>
+</segment>
+</net>
+<net name="BAT_STAT" class="0">
+<segment>
+<wire x1="127" y1="144.78" x2="96.52" y2="144.78" width="0.1524" layer="91"/>
+<label x="96.52" y="144.78" size="1.778" layer="95" rot="R180" xref="yes"/>
+<pinref part="U5" gate="G$1" pin="PC10"/>
+</segment>
+</net>
+<net name="2V8_PGOOD" class="0">
+<segment>
+<wire x1="170.18" y1="119.38" x2="175.26" y2="119.38" width="0.1524" layer="91"/>
+<label x="175.26" y="119.38" size="1.778" layer="95" xref="yes"/>
+<pinref part="U5" gate="G$1" pin="PF3"/>
+</segment>
+</net>
+<net name="EXT_TRIG" class="0">
+<segment>
+<wire x1="170.18" y1="175.26" x2="175.26" y2="175.26" width="0.1524" layer="91"/>
+<label x="175.26" y="175.26" size="1.778" layer="95" xref="yes"/>
+<pinref part="U5" gate="G$1" pin="PB15"/>
+</segment>
+</net>
+<net name="EXT_EN" class="0">
+<segment>
+<wire x1="170.18" y1="177.8" x2="200.66" y2="177.8" width="0.1524" layer="91"/>
+<label x="200.66" y="177.8" size="1.778" layer="95" xref="yes"/>
+<pinref part="U5" gate="G$1" pin="PB14"/>
+</segment>
+</net>
 <net name="RFM_RST" class="0">
+<segment>
+<label x="175.26" y="132.08" size="1.778" layer="95" xref="yes"/>
+<wire x1="170.18" y1="132.08" x2="175.26" y2="132.08" width="0.1524" layer="91"/>
+<pinref part="U5" gate="G$1" pin="PD15"/>
+</segment>
+</net>
+<net name="!RFM_CS" class="0">
 <segment>
 <label x="200.66" y="139.7" size="1.778" layer="95" xref="yes"/>
@@
 </segment>
 </net>
-<net name="!RFM_CS" class="0">
-<segment>
-<label x="175.26" y="137.16" size="1.778" layer="95" xref="yes"/>
-<wire x1="170.18" y1="137.16" x2="175.26" y2="137.16" width="0.1524" layer="91"/>
-<pinref part="U5" gate="G$1" pin="PD13"/>
-</segment>
-</net>
-<net name="US1_CLK" class="0">
-<segment>
-<label x="121.92" y="210.82" size="1.778" layer="95" rot="R180" xref="yes"/>
-<wire x1="127" y1="210.82" x2="121.92" y2="210.82" width="0.1524" layer="91"/>
-<pinref part="U5" gate="G$1" pin="PA1"/>
-</segment>
-</net>
-<net name="US1_MOSI" class="0">
-<segment>
-<label x="96.52" y="213.36" size="1.778" layer="95" rot="R180" xref="yes"/>
-<wire x1="127" y1="213.36" x2="96.52" y2="213.36" width="0.1524" layer="91"/>
-<pinref part="U5" gate="G$1" pin="PA0"/>
-</segment>
-</net>
-<net name="LED_EN" class="0">
-<segment>
-<wire x1="170.18" y1="185.42" x2="175.26" y2="185.42" width="0.1524" layer="91"/>
-<label x="175.26" y="185.42" size="1.778" layer="95" xref="yes"/>
-<pinref part="U5" gate="G$1" pin="PB11"/>
-</segment>
-</net>
-<net name="VBAT_SENSE" class="0">
-<segment>
-<wire x1="127" y1="142.24" x2="121.92" y2="142.24" width="0.1524" layer="91"/>
-<label x="121.92" y="142.24" size="1.778" layer="95" rot="R180" xref="yes"/>
-<pinref part="U5" gate="G$1" pin="PC11"/>
-</segment>
-</net>
-<net name="BAT_STAT" class="0">
-<segment>
-<wire x1="127" y1="144.78" x2="96.52" y2="144.78" width="0.1524" layer="91"/>
-<label x="96.52" y="144.78" size="1.778" layer="95" rot="R180" xref="yes"/>
-<pinref part="U5" gate="G$1" pin="PC10"/>
-</segment>
-</net>
-<net name="2V8_PGOOD" class="0">
-<segment>
-<wire x1="170.18" y1="119.38" x2="175.26" y2="119.38" width="0.1524" layer="91"/>
-<label x="175.26" y="119.38" size="1.778" layer="95" xref="yes"/>
-<pinref part="U5" gate="G$1" pin="PF3"/>
-</segment>
-</net>
-<net name="EXT_TRIG" class="0">
-<segment>
-<wire x1="170.18" y1="175.26" x2="175.26" y2="175.26" width="0.1524" layer="91"/>
-<label x="175.26" y="175.26" size="1.778" layer="95" xref="yes"/>
-<pinref part="U5" gate="G$1" pin="PB15"/>
-</segment>
-</net>
-<net name="EXT_EN" class="0">
-<segment>
-<wire x1="170.18" y1="177.8" x2="200.66" y2="177.8" width="0.1524" layer="91"/>
-<label x="200.66" y="177.8" size="1.778" layer="95" xref="yes"/>
-<pinref part="U5" gate="G$1" pin="PB14"/>
-</segment>
-</net>

Commit message: Finish board Generate gerbers
Parts:
- added LOGO1: GECKO-14MM, Silkscreen:GECKO-14MM
- added LOGO2: OSHW-LOGOM, Silkscreen:OSHW-LOGOM
Changed lines of the file:
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@@
 <part name="C23" library="Capacitor" deviceset="CAPACITOR" device="-0603" value="1uF"/>
 <part name="GND50" library="Supply Symbol" deviceset="GND" device=""/>
+<part name="LOGO1" library="Silkscreen" deviceset="GECKO" device="-14MM"/>
+<part name="LOGO2" library="Silkscreen" deviceset="OSHW-LOGO" device="M"/>
 </parts>
 <sheets>
@@
 <attribute name="VALUE" x="149.606" y="190.5" size="1.778" layer="96"/>
 </instance>
+<instance part="LOGO1" gate="G$1" x="368.3" y="27.94" smashed="yes"/>
+<instance part="LOGO2" gate="G$1" x="271.78" y="17.78" smashed="yes"/>
 </instances>
 <busses>

Commit message: Fix USB C
Parts:
- USB1: value USB-C-16P-SMD-FLAT-SIDE -> USB-C-16P-SMD-FLAT-SIDE-TYPE-2; device USB Connector:USB-C-16P-SMD-FLAT-SIDE -> USB Connector:USB-C-16P-SMD-FLAT-SIDE-TYPE-2
Changed lines of the file:
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@@
 <part name="VBAT5" library="Supply Symbol" deviceset="VBAT" device=""/>
 <part name="U4" library="Fortune" deviceset="FS8205" device=""/>
-<part name="USB1" library="USB Connector" deviceset="USB-C-16P-SMD-FLAT-SIDE" device=""/>
+<part name="USB1" library="USB Connector" deviceset="USB-C-16P-SMD-FLAT-SIDE" device="-TYPE-2"/>
 <part name="C2" library="Capacitor" deviceset="CAPACITOR" device="-1206" value="100uF"/>
 <part name="R1" library="Resistor" deviceset="RESISTOR" device="-0603" value="5.1K Ohms"/>
